File: Connectors.kicad_sch (KiCad schematic)
At the start: 4 parts, among them J1 Conn_01x09, J2 Conn_01x04, J3 Conn_01x04, J4 Conn_02x03_Odd_Even

Commit message: Schematic Complete
Parts:
- J1: renamed from J2; footprint (none) -> Connector_PinHeader_2.54mm:PinHeader_1x04_P2.54mm_Vertical; Purpose (none) -> I2C
- J2: renamed from J1; footprint (none) -> Connector_PinHeader_2.54mm:PinHeader_1x09_P2.54mm_Vertical; Purpose (none) -> GPIO
- J3: footprint (none) -> Connector_PinHeader_2.54mm:PinHeader_1x04_P2.54mm_Vertical; Purpose (none) -> SERIAL UART
- J4: footprint (none) -> Connector_PinHeader_2.54mm:PinHeader_2x03_P2.54mm_Vertical; Purpose (none) -> ICSP
Connections:
- net D2: now reaches J2.1 (Pin_1)
- net D3: now reaches J2.2 (Pin_2)
- net D4: now reaches J2.3 (Pin_3)
- net D5: now reaches J2.4 (Pin_4)
- net D6: now reaches J2.5 (Pin_5)
- net D7: now reaches J2.6 (Pin_6)
- net D8: now reaches J2.7 (Pin_7)
- net GND: now reaches J2.8 (Pin_8)
- net GND: now also J1.1 (Pin_1), J3.1 (Pin_1), J4.6 (Pin_6)
- net Vcc: now reaches J2.9 (Pin_9)
- net Vcc: now also J1.2 (Pin_2), J3.2 (Pin_2), J4.2 (Pin_2)
- net MISO: now reaches J4.1 (Pin_1)
- net SCK: now reaches J4.3 (Pin_3)
- net MOSI: now reaches J4.4 (Pin_4)
- net RESET: now reaches J4.5 (Pin_5)
- net RX: now reaches J3.3 (Pin_3)
- net TX: now reaches J3.4 (Pin_4)
- net SDA: now reaches J1.3 (Pin_3)
- net SCL: now reaches J1.4 (Pin_4)

Commit message: Schematic ok
Other:
- note added: "Connectors"
- moved on the sheet: J3, J4
Changed lines of the file:
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@@
 	(generator_version "9.0")
 	(paper "A4")
+	(text "Connectors\n"
+		(exclude_from_sim no)
+		(at 58.674 101.854 0)
+		(effects
+			(font
+				(size 2.5 2.5)
+			)
+		)
+	)
 	(hierarchical_label "MOSI"
 		(shape input)
-		(at 130.81 72.39 0)
+		(at 99.06 72.39 0)
 		(effects
 			(font
@@
 	(hierarchical_label "SCK"
 		(shape passive)
-		(at 118.11 72.39 180)
+		(at 86.36 72.39 180)
 		(effects
 			(font
@@
 	(hierarchical_label "GND"
 		(shape passive)
-		(at 130.81 74.93 0)
+		(at 99.06 74.93 0)
 		(effects
 			(font
@@
 	(hierarchical_label "Vcc"
 		(shape passive)
-		(at 120.65 41.91 180)
+		(at 88.9 41.91 180)
 		(effects
 			(font
@@
 	(hierarchical_label "GND"
 		(shape passive)
-		(at 120.65 39.37 180)
+		(at 88.9 39.37 180)
 		(effects
 			(font
@@
 	(hierarchical_label "MISO"
 		(shape output)
-		(at 118.11 69.85 180)
+		(at 86.36 69.85 180)
 		(effects
 			(font
@@
 	(hierarchical_label "Vcc"
 		(shape passive)
-		(at 130.81 69.85 0)
+		(at 99.06 69.85 0)
 		(effects
 			(font
@@
 	(hierarchical_label "RX"
 		(shape input)
-		(at 120.65 44.45 180)
+		(at 88.9 44.45 180)
 		(effects
 			(font
@@
 	(hierarchical_label "TX"
 		(shape output)
-		(at 120.65 46.99 180)
+		(at 88.9 46.99 180)
 		(effects
 			(font
@@
 	(hierarchical_label "RESET"
 		(shape passive)
-		(at 118.11 74.93 180)
+		(at 86.36 74.93 180)
 		(effects
 			(font
@@
 			)
 			(justify right)
+		)
+	)
+	(rule_area
+		(polyline
+			(pts
+				(xy 48.26 34.29) (xy 109.22 34.29) (xy 109.22 97.79) (xy 48.26 97.79)
+			)
+			(stroke
+				(width 0.3)
+				(type dash)
+				(color 0 0 194 1)
+			)
+			(fill
+				(type none)
+			)
 		)
 	)
@@
 	(symbol
 		(lib_id "Connector_Generic:Conn_02x03_Odd_Even")
-		(at 123.19 72.39 0)
+		(at 91.44 72.39 0)
 		(unit 1)
 		(exclude_from_sim no)
@@
 		(dnp no)
 		(property "Reference" "J4"
-			(at 124.46 63.5 0)
+			(at 92.71 63.5 0)
 			(effects
 				(font
@@
 		)
 		(property "Value" "Conn_02x03_Odd_Even"
-			(at 124.46 66.04 0)
+			(at 92.71 66.04 0)
 			(effects
 				(font
@@
 		)
 		(property "Footprint" "Connector_PinHeader_2.54mm:PinHeader_2x03_P2.54mm_Vertical"
-			(at 123.19 72.39 0)
+			(at 91.44 72.39 0)
 			(effects
 				(font
@@
 		)
 		(property "Datasheet" "~"
-			(at 123.19 72.39 0)
+			(at 91.44 72.39 0)
 			(effects
 				(font
@@
 		)
 		(property "Description" "Generic connector, double row, 02x03, odd/even pin numbering scheme (row 1 odd numbers, row 2 even numbers), script generated (kicad-library-utils/schlib/autogen/connector/)"
-			(at 123.19 72.39 0)
+			(at 91.44 72.39 0)
 			(effects
 				(font
@@
 		)
 		(property "Sim.Device" ""
-			(at 123.19 72.39 0)
+			(at 91.44 72.39 0)
 			(effects
 				(font
@@
 		)
 		(property "Purpose" "ICSP"
-			(at 124.714 78.232 0)
+			(at 92.964 78.232 0)
 			(effects
 				(font
@@
 	(symbol
 		(lib_id "Connector_Generic:Conn_01x04")
-		(at 125.73 41.91 0)
+		(at 93.98 41.91 0)
 		(unit 1)
 		(exclude_from_sim no)
@@
 		(dnp no)
 		(property "Reference" "J3"
-			(at 128.27 41.9099 0)
+			(at 96.52 41.9099 0)
 			(effects
 				(font
@@
 		)
 		(property "Value" "Conn_01x04"
-			(at 128.27 44.4499 0)
+			(at 96.52 44.4499 0)
 			(effects
 				(font
@@
 		)
 		(property "Footprint" "Connector_PinHeader_2.54mm:PinHeader_1x04_P2.54mm_Vertical"
-			(at 125.73 41.91 0)
+			(at 93.98 41.91 0)
 			(effects
 				(font
@@
 		)
 		(property "Datasheet" "~"
-			(at 125.73 41.91 0)
+			(at 93.98 41.91 0)
 			(effects
 				(font
@@
 		)
 		(property "Description" "Generic connector, single row, 01x04, script generated (kicad-library-utils/schlib/autogen/connector/)"
-			(at 125.73 41.91 0)
+			(at 93.98 41.91 0)
 			(effects
 				(font
@@
 		)
 		(property "Sim.Device" ""
-			(at 125.73 41.91 0)
+			(at 93.98 41.91 0)
 			(effects
 				(font
@@
 		)
 		(property "Purpose" "SERIAL UART"
-			(at 125.73 51.054 0)
-			(effects
-				(font
+			(at 93.98 51.054 0)
+			(effects
+				(font
