File: Connectors.kicad_sch (KiCad schematic)
At the start: 5 parts, among them J1 Conn_01x04, J2 Conn_01x09, J3 Conn_02x03_Odd_Even, J4 Conn_01x04, J5 Conn_01x07

Commit message: Complete 2-layer pcb
Parts:
- renumbered J1 to J3, J3 to J4, J2 to J5, J4 to J6, J5 to J7
Changed lines of the file:
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@@
 		(on_board yes)
 		(dnp no)
-		(property "Reference" "J2"
+		(property "Reference" "J5"
 			(at 64.77 78.7399 0)
 			(effects
@@
 			(project ""
 				(path "/a08b1d3f-e118-4ee7-8d96-2e220d0668f8/d051774b-47dc-4f71-a75f-a0885941fe0a"
-					(reference "J2")
+					(reference "J5")
 					(unit 1)
 				)
@@
 		(on_board yes)
 		(dnp no)
-		(property "Reference" "J3"
+		(property "Reference" "J4"
 			(at 63.5 52.07 0)
 			(effects
@@
 			(project ""
 				(path "/a08b1d3f-e118-4ee7-8d96-2e220d0668f8/d051774b-47dc-4f71-a75f-a0885941fe0a"
-					(reference "J3")
+					(reference "J4")
 					(unit 1)
 				)
@@
 		(on_board yes)
 		(dnp no)
-		(property "Reference" "J4"
+		(property "Reference" "J6"
 			(at 96.52 41.9099 0)
 			(effects
@@
 			(project "MCU_Datalogger"
 				(path "/a08b1d3f-e118-4ee7-8d96-2e220d0668f8/d051774b-47dc-4f71-a75f-a0885941fe0a"
-					(reference "J4")
+					(reference "J6")
 					(unit 1)
 				)
@@
 		(on_board yes)
 		(dnp no)
-		(property "Reference" "J1"
+		(property "Reference" "J3"
 			(at 64.77 41.9099 0)
 			(effects
@@
 			(project ""
 				(path "/a08b1d3f-e118-4ee7-8d96-2e220d0668f8/d051774b-47dc-4f71-a75f-a0885941fe0a"
-					(reference "J1")
+					(reference "J3")
 					(unit 1)
 				)
@@
 		(dnp no)
 		(fields_autoplaced yes)
-		(property "Reference" "J5"
+		(property "Reference" "J7"
 			(at 96.52 81.2799 0)
 			(effects
@@
 			(project ""
 				(path "/a08b1d3f-e118-4ee7-8d96-2e220d0668f8/d051774b-47dc-4f71-a75f-a0885941fe0a"
-					(reference "J5")
+					(reference "J7")
 					(unit 1)
 				)
