File: MCU_Datalogger.kicad_pcb (KiCad board)
At the start: 2 copper layers, 29 parts, among them J1 Conn_01x04, J2 Conn_01x09, J3 Conn_01x04, J4 Conn_02x03_Odd_Even, U1 ATMEGA328P-AU, U2 DS1337S_, U3 24LC1025, U4 24LC1025, Y1 32.768 KHz, Y2 16 MHz

Commit message: Some changes to the original design of the kicad book
Parts:
- removed BT1: Battery, Connector_PinHeader_2.54mm:PinHeader_1x02_P2.54mm_Vertical
- removed the R2 at (135.2, 79.8)
- added C1: 10pF, Capacitor_SMD:C_0805_2012Metric, F.Cu at (144.8, 58.1)
- added C2: 10pF, Capacitor_SMD:C_0805_2012Metric, F.Cu at (144.8, 61.1)
- added C3: 100pF, Capacitor_SMD:C_0805_2012Metric, F.Cu at (144.8, 64.1)
- added D1: BAT54J, Diode_SMD:D_SOD-323F, F.Cu at (149.2, 61.0)
- added J5: Conn_01x07, Connector_PinHeader_2.54mm:PinHeader_1x07_P2.54mm_Vertical, F.Cu at (156.7, 52.4)
- added J6: S8411-45R, S8411-45R:HARWIN_S8411-45R, F.Cu at (134.5, 61.5)
- added J7: USB_B_Micro, digikey-footprints:USB_Micro_B_Female_6pin, F.Cu at (147.5, 52.4)
- added R1: 1k, Resistor_SMD:R_0805_2012Metric, F.Cu at (149.3, 58.1)
- R2: renamed from R1; value 10K -> 4.7K
- U2: value DS1337S_ -> MCP7940NT-I_SN; footprint DS1337S_:SOIC127P600X175-8N -> MCP7940N_SOIC:SOIC127P600X175-8N
- Y1: footprint Crystal:Crystal_SMD_5032-2Pin_5.0x3.2mm_HandSoldering -> FC-135_32.7680KA-A0:XTAL_FC-135_32.7680KA-A0
- moved U2 35.3 mm to (147.4, 68.8)
- moved H1 26.7 mm to (123.5, 52.3)
- moved H2 26.7 mm to (123.5, 58.0)
- moved H3 26.7 mm to (123.5, 63.8)
- moved H4 26.7 mm to (123.5, 69.5)
- moved J1 25.6 mm to (166.3, 52.0)
- moved J2 25.6 mm to (161.6, 52.0)
- moved J3 25.6 mm to (166.3, 64.3)
- moved J4 25.6 mm to (170.9, 52.0)
- moved C4 23.5 mm to (170.1, 76.8)
- moved C8 22.1 mm to (165.2, 85.7)
- moved D3 22.1 mm to (169.7, 83.9)
- moved C5 22.1 mm to (165.2, 76.7)
- moved C6 22.1 mm to (165.2, 79.7)
- moved C7 22.1 mm to (165.2, 82.7)
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- renumbered C1 to C4, C2 to C5, C3 to C6, C4 to C7, C5 to C8, D1 to D2, D2 to D3, J4 to J3, J3 to J4, U3 to U1, U4 to U3, U1 to U4
Connections:
- net Net-(U1-AREF) renamed /AREF
- C8 pad 1: Net-(BT1-+) -> /Vcc
- D3 pad 2: Net-(BT1-+) -> /Vcc
- J2 pad 1: /D2 -> GND
- J2 pad 8: GND -> /B1
- J2 pad 9: /Vcc -> /B2/SS
- R2 pad 2: Net-(U2-~{INTA}) -> /MFP
- U2 pad 3: Net-(U2-~{INTA}) -> Net-(U2-VBAT)
- U2 pad 7: Net-(U2-SQW/~INT) -> /MFP
- U4 pad 13: unconnected-(U1-PB1-Pad13) -> /B1
- U4 pad 14: unconnected-(U1-PB2-Pad14) -> /B2/SS
- U4 pad 18: Net-(BT1-+) -> /Vcc
- U4 pad 19: unconnected-(U1-ADC6-Pad19) -> /ADC6
- U4 pad 22: unconnected-(U1-ADC7-Pad22) -> /ADC7
- U4 pad 23: unconnected-(U1-PC0-Pad23) -> /ADC0
- U4 pad 24: unconnected-(U1-PC1-Pad24) -> /ADC1
- U4 pad 25: unconnected-(U1-PC2-Pad25) -> /ADC2
- U4 pad 26: unconnected-(U1-PC3-Pad26) -> /ADC3
- U4 pad 32: /D2 -> /MFP
- U4 pad 4: Net-(BT1-+) -> /Vcc
- U4 pad 6: unconnected-(U1-VCC-Pad6) -> /Vcc

Commit message: Complete 2-layer pcb
Parts:
- removed D3: LED, LED_SMD:LED_0805_2012Metric
- added C10: 100nF, Capacitor_SMD:C_0805_2012Metric, F.Cu at (96.1, 89.1)
- added C11: 10uF, Capacitor_SMD:C_0805_2012Metric, F.Cu at (83.1, 66.2)
- added C12: 100nF, Capacitor_SMD:C_0805_2012Metric, F.Cu at (107.7, 62.8)
- added C13: 100nF, Capacitor_SMD:C_0805_2012Metric, F.Cu at (120.0, 65.9)
- added C9: 100nF, Capacitor_SMD:C_0805_2012Metric, F.Cu at (93.1, 78.3)
- added REF**: KiCad-Logo2_6mm_SilkScreen, Symbol:KiCad-Logo2_6mm_SilkScreen, B.Cu at (80.0, 69.3)
- J1: value Conn_01x04 -> S8411-45R; footprint Connector_PinHeader_2.54mm:PinHeader_1x04_P2.54mm_Vertical -> S8411-45R:HARWIN_S8411-45R
- J2: value Conn_01x09 -> USB_B_Micro; footprint Connector_PinHeader_2.54mm:PinHeader_1x09_P2.54mm_Vertical -> digikey-footprints:USB_Micro_B_Female_6pin
- J3: value Conn_02x03_Odd_Even -> Conn_01x04; footprint Connector_PinHeader_2.54mm:PinHeader_2x03_P2.54mm_Vertical -> Connector_PinHeader_2.54mm:PinHeader_1x04_P2.54mm_Vertical
- J4: value Conn_01x04 -> Conn_02x03_Odd_Even; footprint Connector_PinHeader_2.54mm:PinHeader_1x04_P2.54mm_Vertical -> Connector_PinHeader_2.54mm:PinHeader_2x03_P2.54mm_Vertical
- J5: value Conn_01x07 -> Conn_01x09; footprint Connector_PinHeader_2.54mm:PinHeader_1x07_P2.54mm_Vertical -> Connector_PinHeader_2.54mm:PinHeader_1x09_P2.54mm_Vertical
- J6: value S8411-45R -> Conn_01x04; footprint S8411-45R:HARWIN_S8411-45R -> Connector_PinHeader_2.54mm:PinHeader_1x04_P2.54mm_Vertical
- J7: value USB_B_Micro -> Conn_01x07; footprint digikey-footprints:USB_Micro_B_Female_6pin -> Connector_PinHeader_2.54mm:PinHeader_1x07_P2.54mm_Vertical
- R5: value 330 -> 10K
- R6: value 10K -> 330
- R7: value 330 -> 10
- moved J1 92.3 mm to (78.3, 80.2)
- moved J2 79.3 mm to (82.8, 60.8)
- moved C6 77.4 mm to (88.2, 87.1)
- moved C5 77.2 mm to (88.2, 81.9)
- moved J5 73.8 mm to (95.0, 92.8), turned to 90 degrees
- moved D1 73.7 mm to (82.5, 92.4), turned to 180 degrees
- moved R1 71.7 mm to (86.3, 92.4), turned to 180 degrees
- moved C4 70.9 mm to (100.1, 66.1)
- moved Y2 66.7 mm to (91.9, 84.5)
- moved J4 66.3 mm to (115.4, 88.4), turned to 90 degrees
- moved Y1 64.8 mm to (91.4, 68.8), turned to 90 degrees
- moved H2 63.0 mm to (71.6, 93.7)
- moved C7 56.9 mm to (108.4, 80.4), turned to 90 degrees
- moved C2 55.5 mm to (90.4, 72.0)
- moved C8 55.4 mm to (109.9, 84.0)
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Connections:
- C8 pad 1: /Vcc -> Net-(U4-AVCC)
- D2 pad 2: /SCK -> /Vcc
- J2 pad 1: GND -> /Vcc
- J2 pad 2: /D3 -> unconnected-(J2-D--Pad2)
- J2 pad 3: /D4 -> unconnected-(J2-D+-Pad3)
- J2 pad 4: /D5 -> unconnected-(J2-ID-Pad4)
- J2 pad 5: /D6 -> GND
- J2 pad 6: /D7 -> GND
- J3 pad 1: /MISO -> GND
- J3 pad 3: /SCK -> /SDA
- J3 pad 4: /MOSI -> /SCL
- J4 pad 1: GND -> /MISO
- J4 pad 3: /RX -> /SCK
- J4 pad 4: /TX -> /MOSI
- J5 pad 1: /ADC0 -> GND
- J5 pad 2: /ADC1 -> /D3
- J5 pad 3: /ADC2 -> /D4
- J5 pad 4: /ADC3 -> /D5
- J5 pad 5: /ADC6 -> /D6
- J5 pad 6: /ADC7 -> /D7
- J5 pad 7: /AREF -> /D8
- J7 pad 1: /Vcc -> /ADC0
- J7 pad 2: unconnected-(J7-D--Pad2) -> /ADC1
- J7 pad 3: unconnected-(J7-D+-Pad3) -> /ADC2
- J7 pad 4: unconnected-(J7-ID-Pad4) -> /ADC3
- J7 pad 5: GND -> /ADC6
- J7 pad 6: GND -> /ADC7
- R5 pad 1: GND -> /Vcc
- R5 pad 2: Net-(D2-K) -> /RESET
- R6 pad 1: /Vcc -> Net-(D2-K)
- R6 pad 2: /RESET -> GND
- R7 pad 1: Net-(D3-K) -> Net-(U4-AVCC)
- R7 pad 2: GND -> /Vcc
- U4 pad 18: /Vcc -> Net-(U4-AVCC)
Routing:
- net /Vcc: track 0.00 -> 192.5 mm, vias 0 -> 9
- net /SDA: track 0.00 -> 55.2 mm
- net /SCL: track 0.00 -> 50.1 mm
- net /RESET: track 0.00 -> 46.8 mm, vias 0 -> 2
- net Net-(U2-VBAT): track 0.00 -> 35.4 mm, vias 0 -> 2
- net /ADC3: track 0.00 -> 26.8 mm, vias 0 -> 2
- net /AREF: track 0.00 -> 26.6 mm, vias 0 -> 2
- net /ADC2: track 0.00 -> 26.4 mm
- net /ADC0: track 0.00 -> 25.9 mm, vias 0 -> 2
- net /ADC6: track 0.00 -> 25.8 mm, vias 0 -> 2
- net /MOSI: track 0.00 -> 24.2 mm
- net /ADC7: track 0.00 -> 23.6 mm, vias 0 -> 2
- net /ADC1: track 0.00 -> 22.8 mm, vias 0 -> 4
- net /TX: track 0.00 -> 17.5 mm, vias 0 -> 1
- net /B2/SS: track 0.00 -> 17.3 mm
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- added copper zone on B.Cu, net GND
- added copper zone on F.Cu, net GND
Other:
- board outline added: 60.8 x 39.2 mm
- board text added: "-2 MBIT EEPROM -RTC -I2C, SPI"
- board text added: "A0"
- board text added: "A1"
- board text added: "A2"
- board text added: "A3"
- board text added: "A6"
- board text added: "A7"
- board text added: "AREF"
- board text added: "B1"
- board text added: "B2"
- board text added: "D3"
- board text added: "D4"
- board text added: "D5"
- board text added: "D6"
- board text added: "D7"
- board text added: "D8"
- board text added: "Data Logger ATMega328"
- board text added: "GND"
- board text added: "I2C"
- board text added: "ICSP"
- board text added: "ICSP MISO | VCC SCK | MOSI RESET| GND"
- board text added: "RX"
- board text added: "SCL"
- board text added: "SDA"
- board text added: "SERIAL"
- board text added: "TX"
- board text added: "VCC"
