File: MCU_Datalogger.kicad_sch (KiCad schematic)
At the start: 30 parts, among them J6 S8411-45R, J7 USB_B_Micro, U1 24LC1025, U2 MCP7940NT-I_SN, U3 24LC1025, U4 ATMEGA328P-AU, Y1 32.768 KHz, Y2 16 MHz

Commit message: Complete 2-layer pcb
Parts:
- removed D2: LED, LED_SMD:LED_0805_2012Metric, symbol Device:LED
- removed R5: 330, Resistor_SMD:R_0805_2012Metric, symbol Device:R_US
- added C10, C12, C13, C9: 100nF, Capacitor_SMD:C_0805_2012Metric, symbol Device:C
- added C11: 10uF, Capacitor_SMD:C_0805_2012Metric, symbol Device:C
- added R7: 10, Resistor_SMD:R_0805_2012Metric, symbol Device:R_US
- renumbered D3 to D2, J6 to J1, J7 to J2, R6 to R5, R7 to R6
Connections:
- net GND: now also C10.2, C11.2, C12.1, C13.2, C9.2
- net Vcc: now also C10.1, C11.1, C12.2, C13.1, C9.1, R7.2; no longer C8.1, U4.18 (AVCC)
- new net: C8.1, R7.1, U4.18 (AVCC)
Other:
- moved on the sheet: C5, C6, C7, C8, D2, J2, R5, R6, U4, Y2
